Commit message: first commit

File: urdf/robotiq_85_gripper.transmission.xacro (robot description, xacro)
@@ -5,14 +5,14 @@
             <type>transmission_interface/SimpleTransmission</type>
             <joint name="${prefix}robotiq_85_left_knuckle_joint">
-                <hardwareInterface>EffortJointInterface</hardwareInterface>
+                <hardwareInterface>hardware_interface/PositionJointInterface</hardwareInterface>
             </joint>
             <actuator name="${prefix}robotiq_85_left_knuckle_motor">
                 <mechanicalReduction>1</mechanicalReduction>
-                <hardwareInterface>EffortJointInterface</hardwareInterface>
+                <hardwareInterface>hardware_interface/PositionJointInterface</hardwareInterface>
             </actuator>
         </transmission>
         <gazebo>
                 <!-- loading plugin: mimic joints works in gazebo now -->
-            <plugin filename="libroboticsgroup_gazebo_mimic_joint_plugin.so" name="${prefix}mimic_robotiq_85_1">
+            <plugin filename="libroboticsgroup_upatras_gazebo_mimic_joint_plugin.so" name="${prefix}mimic_robotiq_85_1">
                 <joint>${prefix}robotiq_85_left_knuckle_joint</joint>
                 <mimicJoint>${prefix}robotiq_85_right_knuckle_joint</mimicJoint>
@@ -20,5 +20,5 @@
                 <offset>0.0</offset-->
             </plugin>
-            <plugin filename="libroboticsgroup_gazebo_mimic_joint_plugin.so" name="${prefix}mimic_robotiq_85_2">
+            <plugin filename="libroboticsgroup_upatras_gazebo_mimic_joint_plugin.so" name="${prefix}mimic_robotiq_85_2">
                 <joint>${prefix}robotiq_85_left_knuckle_joint</joint>
                 <mimicJoint>${prefix}robotiq_85_left_inner_knuckle_joint</mimicJoint>
@@ -26,5 +26,5 @@
                 <offset>0.0</offset-->
             </plugin>
-            <plugin filename="libroboticsgroup_gazebo_mimic_joint_plugin.so" name="${prefix}mimic_robotiq_85_3">
+            <plugin filename="libroboticsgroup_upatras_gazebo_mimic_joint_plugin.so" name="${prefix}mimic_robotiq_85_3">
                 <joint>${prefix}robotiq_85_left_knuckle_joint</joint>
                 <mimicJoint>${prefix}robotiq_85_right_inner_knuckle_joint</mimicJoint>
@@ -32,5 +32,5 @@
                 <offset>0.0</offset-->
             </plugin>
-            <plugin filename="libroboticsgroup_gazebo_mimic_joint_plugin.so" name="${prefix}mimic_robotiq_85_4">
+            <plugin filename="libroboticsgroup_upatras_gazebo_mimic_joint_plugin.so" name="${prefix}mimic_robotiq_85_4">
                 <joint>${prefix}robotiq_85_left_knuckle_joint</joint>
                 <mimicJoint>${prefix}robotiq_85_left_finger_tip_joint</mimicJoint>
@@ -38,5 +38,5 @@
                 <!--offset>0.0</offset-->
             </plugin>
-            <plugin filename="libroboticsgroup_gazebo_mimic_joint_plugin.so" name="${prefix}mimic_robotiq_85_5">
+            <plugin filename="libroboticsgroup_upatras_gazebo_mimic_joint_plugin.so" name="${prefix}mimic_robotiq_85_5">
                 <joint>${prefix}robotiq_85_left_knuckle_joint</joint>
                 <mimicJoint>${prefix}robotiq_85_right_finger_tip_joint</mimicJoint>

File: urdf/robotiq_85_gripper.urdf.xacro (robot description, xacro)
@@ -3,10 +3,9 @@
     <xacro:include filename="$(find robotiq_gripper)/urdf/robotiq_85_gripper.transmission.xacro" />
     <xacro:property name="pi" value="3.14159"/>
-    <xacro:macro name="robotiq_85_gripper" params="prefix parent origin_xyz origin_rpy">
-    <!--<xacro:macro name="robotiq_85_gripper" params="prefix parent *origin">-->
+    <xacro:macro name="robotiq_85_gripper" params="prefix parent *origin">
         <joint name="${prefix}robotiq_85_base_joint" type="fixed">
             <parent link="${parent}"/>
             <child link="${prefix}robotiq_85_base_link"/>
-            <origin xyz = "${origin_xyz}" rpy = "${origin_rpy}" />
+            <xacro:insert_block name="origin"/>
         </joint>
         <link name="${prefix}robotiq_85_base_link">

File: urdf/robotiq_85_gripper2.xacro (robot description, xacro)
@@ -7,6 +7,5 @@
     </gazebo>
     <link name="world"/>
-    <xacro:robotiq_85_gripper prefix="" parent="world" >
-        <origin xyz="0.0 0 0.0" rpy="0 0 0"/>
+    <xacro:robotiq_85_gripper prefix="" parent="world" origin_xyz="0 0 0" origin_rpy="0 0 0" >
     </xacro:robotiq_85_gripper>
 </robot>
